Commit message: Updated tms_robot_description and make ready for hardware launch. - bringup.launch.py for running mock version - all.launch.py for real robot and sensor hardware

File: tms_robot_description/urdf/tms_env.xacro (robot description, xacro)
@@ -5,4 +5,5 @@
     <xacro:property name="table_length" value="0.730" /> <!-- x direction -->
     <xacro:property name="table_height" value="0.710" />
+    <xacro:property name="plate_thickness" value="0.010" />
     <xacro:property name="table_dummy_head_offset" value="0.265" /> <!-- to be determined -->
     <xacro:property name="table_ur_offset" value="-0.2025" />
@@ -18,4 +19,19 @@
         <geometry>
           <box size="${table_length} ${table_width} ${table_height}"/>
+        </geometry>
+        <origin rpy="0 0 0" xyz="0 0 0"/>
+      </collision>
+    </link>
+    <link name="robot_mounting_plate">
+      <visual>
+        <geometry>
+          <box size="0.2 0.2 ${plate_thickness}"/>
+        </geometry>
+        <origin rpy="0 0 0" xyz="0 0 0"/>
+        <material name="white"/>
+      </visual>
+      <collision>
+        <geometry>
+          <box size="0.2 0.2 ${plate_thickness}"/>
         </geometry>
         <origin rpy="0 0 0" xyz="0 0 0"/>
@@ -43,8 +59,13 @@
       <origin xyz="0 0 ${table_height/2}" rpy="0 0 0" />
     </joint>
-    <joint name="table_to_robot_mount" type="fixed">
+    <joint name="table_to_robot_mounting_plate" type="fixed">
       <parent link="table"/>
+      <child link="robot_mounting_plate"/>
+      <origin xyz="${table_ur_offset} 0 ${table_height/2+plate_thickness/2}" rpy="0 0 0" />
+    </joint>
+    <joint name="robot_mounting_head" type="fixed">
+      <parent link="robot_mounting_plate"/>
       <child link="robot_mount"/>
-      <origin xyz="${table_ur_offset} 0 ${table_height/2}" rpy="0 0 ${pi}" />
+      <origin xyz="0 0 ${plate_thickness/2}" rpy="0 0 ${pi}" />
     </joint>
     <joint name="table_to_dummy_head" type="fixed">
